File: fabrication/kicad/index.kicad_pcb (KiCad board)
At the start: 4 copper layers, 100 x 124 mm, 141 parts

Commit message: Bundle exact footprint library and require zero DRC violations
Parts:
- ?: footprint tscircuit:Unknown -> tscircuit:g350_mechanical_00cc84886ae3edb8296ba0084244d238
- ?: footprint tscircuit:Unknown -> tscircuit:g350_mechanical_126df3c06cea520113bd683e6b9add83
- ?: footprint tscircuit:Unknown -> tscircuit:g350_mechanical_12f762ea55789b16421766ea26589716
- ?: footprint tscircuit:Unknown -> tscircuit:g350_mechanical_151630806a4215411665a4fe68f2a0c3
- ?: footprint tscircuit:Unknown -> tscircuit:g350_mechanical_176a326021c808012c25dda23683b343
- ?: footprint tscircuit:Unknown -> tscircuit:g350_mechanical_271173c03cd2863f529398be6854ab3d
- ?: footprint tscircuit:Unknown -> tscircuit:g350_mechanical_2714c6c05992f37f25c552425ae267fd
- ?: footprint tscircuit:smtpad_circle_diameter1mm -> tscircuit:g350_mechanical_2a20550a6b7d336a5325ee3611c90fd6
- ?: footprint tscircuit:Unknown -> tscircuit:g350_mechanical_2bb693a02eb9aa4176d617de1c65d9fd
- ?: footprint tscircuit:Unknown -> tscircuit:g350_mechanical_318a99804f1d20bf303b2502506c953d
- ?: footprint tscircuit:Unknown -> tscircuit:g350_mechanical_34e1b998287937b81c10b5d80fa833f8
- ?: footprint tscircuit:Unknown -> tscircuit:g350_mechanical_0377c7aa746fe64a1a97fb165660238a
- ?: footprint tscircuit:Unknown -> tscircuit:g350_mechanical_35765fc02b188a1f20bab47e165cdedd
- ?: footprint tscircuit:Unknown -> tscircuit:g350_mechanical_35a0bdc04b06fc7f345149424c5670fd
- ?: footprint tscircuit:Unknown -> tscircuit:g350_mechanical_38f5384043530de14db0e382580eb923
- ?: footprint tscircuit:Unknown -> tscircuit:g350_mechanical_404ff7404057c2ff3f0082c241a7377d
- ?: footprint tscircuit:Unknown -> tscircuit:g350_mechanical_41a970a04c07464156651be260c2f183
- ?: footprint tscircuit:Unknown -> tscircuit:g350_mechanical_43f892604e56680158b43da263121343
- ?: footprint tscircuit:Unknown -> tscircuit:g350_mechanical_462d578e25831ab26ecc730e031c00ce
- ?: footprint tscircuit:Unknown -> tscircuit:g350_mechanical_46829eae782082f236c3a4920a9939ce
- ?: footprint tscircuit:Unknown -> tscircuit:g350_mechanical_46fac35e3a92417e2e29bf9e21c13dbe
- ?: footprint tscircuit:smtpad_circle_diameter1mm -> tscircuit:g350_mechanical_48d251205e93639f7454761e75ea7763
- ?: footprint tscircuit:Unknown -> tscircuit:g350_mechanical_04a51060110d92401d76142029de9600
- ?: footprint tscircuit:Unknown -> tscircuit:g350_mechanical_4926e8a0114955416bb9932239d62efd
- ?: footprint tscircuit:smtpad_circle_diameter1mm -> tscircuit:g350_mechanical_4a877526092a96c63832479a798f25fa
- ?: footprint tscircuit:hole_circle_holeDiameter2.7mm -> tscircuit:g350_mechanical_4fddb506189248fa7efdb906168dbb06
- ?: footprint tscircuit:hole_circle_holeDiameter2.75mm -> tscircuit:g350_mechanical_504f5d741b6114cc78ee78f40d3e06b4
- ?: footprint tscircuit:Unknown -> tscircuit:g350_mechanical_506d44c02eeb010151bcb93e2d9b8c83
- ?: footprint tscircuit:Unknown -> tscircuit:g350_mechanical_50e3e5865d4c676669b4e946761d6b26
- ?: footprint tscircuit:Unknown -> tscircuit:g350_mechanical_5145b86046e7e2bf3c8a0d1e322c377d
- ?: footprint tscircuit:Unknown -> tscircuit:g350_mechanical_52393ba00837024162a7402242e881fd
- ?: footprint tscircuit:Unknown -> tscircuit:g350_mechanical_5928e8aa17cc0a4a2990d4166aedb276
- ?: footprint tscircuit:smtpad_circle_diameter1mm -> tscircuit:g350_mechanical_5a51f674480f470c158f7b74732e3df4
- ?: footprint tscircuit:Unknown -> tscircuit:g350_mechanical_06df6e20483c4c807666d5203509f6c0
- ?: footprint tscircuit:Unknown -> tscircuit:g350_mechanical_5ad291002485b4c15c22057e23364043
- ?: footprint tscircuit:hole_circle_holeDiameter2.75mm -> tscircuit:g350_mechanical_5be1d5e024c5e45f5a926162261558dd
- ?: footprint tscircuit:Unknown -> tscircuit:g350_mechanical_5e2e28261cd149c6248b949a65e872fa
- ?: footprint tscircuit:smtpad_circle_diameter1mm -> tscircuit:g350_mechanical_61182492037962125a25606e483bdd12
- ?: footprint tscircuit:Unknown -> tscircuit:g350_mechanical_683eb8a01869019f66ef442219b8761d
- ?: footprint tscircuit:Unknown -> tscircuit:g350_mechanical_6bcc21c014db987f6a7cad42162b0cfd
- ?: footprint tscircuit:Unknown -> tscircuit:g350_mechanical_6e134a64263c435c45742ee44edb5edc
- ?: footprint tscircuit:hole_circle_holeDiameter2.7mm -> tscircuit:g350_mechanical_775c9dc02e33245f2c3d19827952a89d
- ?: footprint tscircuit:Unknown -> tscircuit:g350_mechanical_782c0ff46bc38e145f5b0c3452f28a54
- ?: footprint tscircuit:hole_circle_holeDiameter2.75mm -> tscircuit:g350_mechanical_7965eb340db578f45dfaf94c36549474
- ?: footprint tscircuit:smtpad_circle_diameter1mm -> tscircuit:g350_mechanical_09621c201f232e9f34e4411e4aa5539d
- ?: footprint tscircuit:hole_circle_holeDiameter2.7mm -> tscircuit:g350_mechanical_7a8b3ee0201b00ff3a553ce26b3a853d
- ?: footprint tscircuit:hole_circle_holeDiameter2.7mm -> tscircuit:g350_mechanical_7ae5c08078b1bda06c493bc05fe0b9e0
- ?: footprint tscircuit:Unknown -> tscircuit:g350_mechanical_01edb94a3f6f25167f33fc8a3dd71e2a
- ?: footprint tscircuit:Unknown -> tscircuit:g350_mechanical_03ace75a3daff7067f0cd5663f964c3a
- ?: footprint tscircuit:Unknown -> tscircuit:g350_mechanical_0751260048ae046075f51d4034983ee0
- ?: footprint tscircuit:Unknown -> tscircuit:g350_mechanical_07dd36a455c18bdc4c9fb1a410ff10dc
- ?: footprint tscircuit:Unknown -> tscircuit:g350_mechanical_0a79efa0001c19ff0a41bba2149f9143
- ?: footprint tscircuit:Unknown -> tscircuit:g350_mechanical_0be1c9c0665207a13f3dba7e1b328363
- ?: footprint tscircuit:Unknown -> tscircuit:g350_mechanical_122fc2c048407b215d4f46fe02df091d
- ?: footprint tscircuit:Unknown -> tscircuit:g350_mechanical_1294c00a062c3e2a063c43b612a4c596
- ?: footprint tscircuit:hole_circle_holeDiameter2.75mm -> tscircuit:g350_mechanical_0bd7a2e07380a2e10d27175e72312e63
- ?: footprint tscircuit:Unknown -> tscircuit:g350_mechanical_14c4e98453ab147c43e4ed84248b107c
- ?: footprint tscircuit:Unknown -> tscircuit:g350_mechanical_1919d56a52969cd641b8f0ea29f78156
- ?: footprint tscircuit:Unknown -> tscircuit:g350_mechanical_1959ac424445163e5e1c2742007d64c2
- ?: footprint tscircuit:Unknown -> tscircuit:g350_mechanical_210315e02b60eb8135bec122401c96c3
- ?: footprint tscircuit:Unknown -> tscircuit:g350_mechanical_2307e1207d781f012817a31e32589ac3
- ?: footprint tscircuit:Unknown -> tscircuit:g350_mechanical_31d3783e256af65e1902747e0c99f29e
- ?: footprint tscircuit:Unknown -> tscircuit:g350_mechanical_35f92e60405704014ab4d9a25512af43
- ?: footprint tscircuit:Unknown -> tscircuit:g350_mechanical_3ca91e20526a309f682b431e7dec559d
- ?: footprint tscircuit:Unknown -> tscircuit:g350_mechanical_3e1523e053d6365f699748de7f585b5d
- ?: footprint tscircuit:Unknown -> tscircuit:g350_mechanical_3e39e9de7f96c83e3f0c5962025084fe
- ?: footprint tscircuit:Unknown -> tscircuit:g350_mechanical_0e3c25201899fac122f7d0622d55a603
- ?: footprint tscircuit:Unknown -> tscircuit:g350_mechanical_3faab19401b22ccc430f0b2c7b941674
- ?: footprint tscircuit:Unknown -> tscircuit:g350_mechanical_433254403c25f1814481c8be3ad67d03
- ?: footprint tscircuit:Unknown -> tscircuit:g350_mechanical_46e262c05ead5f5f043d217e56331c63
- ?: footprint tscircuit:Unknown -> tscircuit:g350_mechanical_57f14f563c5e3e6a2f5233d664fd59ea
- ?: footprint tscircuit:Unknown -> tscircuit:g350_mechanical_5923b97e3b2bd44230849dfe63caefc2
- ?: footprint tscircuit:Unknown -> tscircuit:g350_mechanical_5930dc00013f61e15baf9fc249e0225d
- ?: footprint tscircuit:Unknown -> tscircuit:g350_mechanical_5d9aa9800e15c8c079c63b001a8952c0
- ?: footprint tscircuit:Unknown -> tscircuit:g350_mechanical_5dbc918047d3309f129d0d426d0d4b23
- ?: footprint tscircuit:Unknown -> tscircuit:g350_mechanical_62a8baa01dfeff9f615946221f4e741d
- ?: footprint tscircuit:Unknown -> tscircuit:g350_mechanical_6b2c050c29cf26ac178db7b458ea9614
- ?: footprint tscircuit:Unknown -> tscircuit:g350_mechanical_0f17d2a01b80548027e8d66034515840
- ?: footprint tscircuit:Unknown -> tscircuit:g350_mechanical_6d33e01a352d5d662871651a79efd866
- ?: footprint tscircuit:Unknown -> tscircuit:g350_mechanical_73f01e205e2f0ba1486df92232ace6a3
- ?: footprint tscircuit:Unknown -> tscircuit:g350_mechanical_74342dc0315b945f2914a9827c7b189d
- ?: footprint tscircuit:Unknown -> tscircuit:g350_mechanical_75c5a45e3468c5fe0cf418624e50f6c2
- ?: footprint tscircuit:Unknown -> tscircuit:g350_mechanical_75fdcc8869954aa85d2cc8c850c446e8
- ?: footprint tscircuit:Unknown -> tscircuit:g350_mechanical_779703e61ff8fe1a4876ffe64f19021a
- ?: footprint tscircuit:Unknown -> tscircuit:g350_mechanical_7fe5d402143561c2577b107e3cd47d42
- ?: footprint tscircuit:Unknown -> tscircuit:g350_mechanical_1066c5206ef180a111b6399e6da20c23
- C_AUDIO_BULK: footprint tscircuit:capacitor_cap0805 -> tscircuit:g350_C_AUDIO_BULK_6c8053e0121015ff486027e25d2f9a3d
- C_AUDIO_HF: footprint tscircuit:capacitor_cap0603 -> tscircuit:g350_C_AUDIO_HF_4f8718706f1c09302dbf2ad0139db390
- C_BAT: footprint tscircuit:capacitor_cap0805 -> tscircuit:g350_C_BAT_29456180576258bf27f5ed0258b1cd3d
- C_BOOST_IN: footprint tscircuit:capacitor_cap0805 -> tscircuit:g350_C_BOOST_IN_599053c04f327e1f44d4a87e3a76d2dd
- C_BOOST_OUT1: footprint tscircuit:capacitor_cap1206 -> tscircuit:g350_C_BOOST_OUT1_4c2ad4da72784cc6311b6e6610416ffa
- C_BOOST_OUT2: footprint tscircuit:capacitor_cap1206 -> tscircuit:g350_C_BOOST_OUT2_7361d6200bf66fa174b14a9e0aa6fb23
- C_FEEDFORWARD: footprint tscircuit:capacitor_cap0603 -> tscircuit:g350_C_FEEDFORWARD_22442cc07cb46aa128db577e3194e663
- C_GAUGE: footprint tscircuit:capacitor_cap0603 -> tscircuit:g350_C_GAUGE_6966ebe01740ce5f68177762189042dd
- C_KEYS: footprint tscircuit:capacitor_cap0603 -> tscircuit:g350_C_KEYS_310dea001b4cd781058bc50210354d7d
- C_KEYS_BULK: footprint tscircuit:capacitor_cap0805 -> tscircuit:g350_C_KEYS_BULK_2335aa005c229bc124851e7e5ad32743
- C_LCD_IN: footprint tscircuit:capacitor_cap0603 -> tscircuit:g350_C_LCD_IN_43be1e2016b21fc171225da2346d647d
- C_LCD_OUT: footprint tscircuit:capacitor_cap0603 -> tscircuit:g350_C_LCD_OUT_1fd467c477bb9a3c0f4b9c3c592461c4
- C_SYS: footprint tscircuit:capacitor_cap0805 -> tscircuit:g350_C_SYS_7a0e31a00699889f78bebd2207e8fd1d
- C_USB: footprint tscircuit:capacitor_cap0603 -> tscircuit:g350_C_USB_1f6d01a05feb442120bc761e5e9bcfa3
- J_BAT: footprint tscircuit:1x3_2_54mm_protected_1S_battery_NTC_harness -> tscircuit:g350_J_BAT_109cbfc049d37e215bbc43fe014c061d
- J_LCD: footprint tscircuit:FPC-05F-18PH20 -> tscircuit:g350_J_LCD_5e66dc500a0921b072791fb02516e250
- J_OFF: footprint tscircuit:1x2_2_54mm_slide-switch_harness -> tscircuit:g350_J_OFF_7db4176027dbaabf3294932272fb2efd
- J_PI: footprint tscircuit:2x20_2_54mm_GPIO_ribbon_header -> tscircuit:g350_J_PI_45b957de51d6aa22169953de7f0951de
- J_SPEAKER: footprint tscircuit:1x2_2_54mm_speaker_harness -> tscircuit:g350_J_SPEAKER_3187528028e8eb617ca6d6be223698dd
- J_USB: footprint tscircuit:TYPE-C-31-M-12 -> tscircuit:g350_J_USB_03455d6058205a605304a8a001d65460
- L_BOOST: footprint tscircuit:WPN252012E1R0MT -> tscircuit:g350_L_BOOST_21aba8e07c1be6c12973db5e30fc6283
- R_ALERT_PULL: footprint tscircuit:resistor_res0603 -> tscircuit:g350_R_ALERT_PULL_3358dc60271761817e78609e240822bd
- R_AUDIO_EN: footprint tscircuit:resistor_res0603 -> tscircuit:g350_R_AUDIO_EN_00256ea05a4acf414b44f2de0f2b4b03
- R_AUDIO_PD: footprint tscircuit:resistor_res0603 -> tscircuit:g350_R_AUDIO_PD_59fa59004b95691f0edad4c2694b12a3
- R_CC1: footprint tscircuit:resistor_res0603 -> tscircuit:g350_R_CC1_70956ae034fa573f2575e6a27fe62483
- R_CC2: footprint tscircuit:resistor_res0603 -> tscircuit:g350_R_CC2_2d72f380781cce9f1dac90be3cc3ad23
- R_CHG_PULL: footprint tscircuit:resistor_res0603 -> tscircuit:g350_R_CHG_PULL_77ce73c01d5e35df3d120802687dba1d
- R_EN: footprint tscircuit:resistor_res0603 -> tscircuit:g350_R_EN_452811c03b7fa87f43d89d423ccf1cfd
- R_FB_HI: footprint tscircuit:resistor_res0603 -> tscircuit:g350_R_FB_HI_376c1ee047ec26e138bb935e469cb263
- R_FB_LO: footprint tscircuit:resistor_res0603 -> tscircuit:g350_R_FB_LO_512b3cc02f7c7d7f4fdbc84230cbf1fd
- R_GOOD_PULL: footprint tscircuit:resistor_res0603 -> tscircuit:g350_R_GOOD_PULL_23af180036c125e16ece9c3e145e5e5d
- R_ILIM: footprint tscircuit:resistor_res0603 -> tscircuit:g350_R_ILIM_6d149d601243a8616e6411de10f433e3
- R_ISET: footprint tscircuit:resistor_res0603 -> tscircuit:g350_R_ISET_2db78cc077d8355f1d67f77e3d084663
- R_RESET: footprint tscircuit:resistor_res0603 -> tscircuit:g350_R_RESET_5f48256a52dfa38a467721aa3a0e9fca
- R_TIMER: footprint tscircuit:resistor_res0603 -> tscircuit:g350_R_TIMER_7cb74c4022470e5f38292f826d66929d
- SW_A: footprint tscircuit:TS-1187A-B-A-B -> tscircuit:g350_SW_A_30040da050a3ac9f2eb4992251f3211d
- SW_B: footprint tscircuit:TS-1187A-B-A-B -> tscircuit:g350_SW_B_2c7ea560542914df2b2f30e25578895d
- SW_DOWN: footprint tscircuit:TS-1187A-B-A-B -> tscircuit:g350_SW_DOWN_1cc9908c10610eac03f88ccc086ff514
- SW_LEFT: footprint tscircuit:TS-1187A-B-A-B -> tscircuit:g350_SW_LEFT_7a95308a6e2caeaa61c42cca555baaea
- SW_MENU: footprint tscircuit:TS-1187A-B-A-B -> tscircuit:g350_SW_MENU_0bf74b4074b06eff0aa7d6c275ffe37d
- SW_RIGHT: footprint tscircuit:TS-1187A-B-A-B -> tscircuit:g350_SW_RIGHT_59a93b904d40b9b040d837d0346fb5f0
- SW_SELECT: footprint tscircuit:TS-1187A-B-A-B -> tscircuit:g350_SW_SELECT_126b40ec1ed3c2cc2b3c44ac37a4c68c
- SW_START: footprint tscircuit:TS-1187A-B-A-B -> tscircuit:g350_SW_START_12d33ba06dd47e9f1183c7226f23f31d
- SW_UP: footprint tscircuit:TS-1187A-B-A-B -> tscircuit:g350_SW_UP_748e63866825e1a65bbd5fc64f54dde6
- SW_X: footprint tscircuit:TS-1187A-B-A-B -> tscircuit:g350_SW_X_03628bc07bf5ba0104b2003e7aa64583
- SW_Y: footprint tscircuit:TS-1187A-B-A-B -> tscircuit:g350_SW_Y_2019cbe0608dee5f1eca576261dd62dd
- TP_3V3: footprint tscircuit:test_point -> tscircuit:g350_TP_3V3_28035840326ce5a17322dc7e18b29e9d
- TP_5V: footprint tscircuit:test_point -> tscircuit:g350_TP_5V_76c068802ecf599f2ba0e44279eedddd
- TP_GND: footprint tscircuit:test_point -> tscircuit:g350_TP_GND_78b643e02cd97e3f2d96bfa277f9027d
- U_AUDIO: footprint tscircuit:MAX98357AETE_T -> tscircuit:g350_U_AUDIO_22ebc3c07d5c01a12833c07e323c7d63
- U_BOOST: footprint tscircuit:TPS61023DRLR -> tscircuit:g350_U_BOOST_2abdfbe07ad1c63f2061885e3a0eb583
- U_CHARGE: footprint tscircuit:BQ24074RGTR -> tscircuit:g350_U_CHARGE_49083820116805c16bd843a239b77e7d
- U_GAUGE: footprint tscircuit:MAX17048G_T10 -> tscircuit:g350_U_GAUGE_26e227007ead9b1f243d5d3e3632e0a3
- U_KEYS: footprint tscircuit:MCP23017-E_SO -> tscircuit:g350_U_KEYS_15ba455e0951c37e0316be620f7f4042
- U_LCD_PWR: footprint tscircuit:AP2112K-3_3TRG1 -> tscircuit:g350_U_LCD_PWR_1d604a603d0ff381687fce9e0e0f90bd

Commit message: Release top-only Rev B carrier with shared USB-C charging and data
Parts:
- removed the ? at (117.0, 56.5)
- removed the ? at (128.0, 85.5)
- removed the ? at (124.1, 54.9)
- removed the ? at (119.8, 51.7)
- removed the ? at (105.2, 117.0)
- removed the ? at (138.0, 51.0) (x2)
- removed the ? at (61.0, 60.0)
- removed the ? at (61.0, 140.0)
- removed the ? at (134.5, 82.9)
- removed the ? at (126.3, 74.5)
- removed the ? at (123.0, 60.1)
- removed the ? at (129.2, 83.9)
- removed the ? at (120.0, 100.0)
- removed the ? at (118.5, 54.5)
- removed the ? at (114.8, 48.7)
- removed the ? at (100.0, 45.0)
- removed the ? at (62.0, 51.0) (x2)
- removed the ? at (121.0, 60.0)
- removed the ? at (139.0, 140.0)
- removed the ? at (103.8, 49.5)
- removed the ? at (117.0, 60.0)
- removed the ? at (117.2, 55.7)
- removed the ? at (62.0, 149.0) (x2)
- removed the ? at (103.4, 53.8)
- removed the ? at (107.6, 67.7)
- removed the ? at (109.0, 48.3)
- removed the ? at (112.7, 58.0)
- removed the ? at (139.0, 60.0)
- removed the ? at (95.3, 115.5)
- removed the ? at (125.7, 69.3)
- removed the ? at (126.7, 44.0)
- removed the ? at (101.2, 104.6)
- removed the ? at (109.5, 116.0)
- removed the ? at (96.0, 123.0)
- removed the ? at (82.0, 113.0)
- removed the ? at (67.0, 76.3)
- removed the ? at (66.0, 84.0)
- removed the ? at (67.7, 83.4)
- removed the ? at (105.7, 110.6)
- removed the ? at (68.6, 82.8)
- removed the ? at (82.0, 104.0)
- removed the ? at (67.0, 78.8)
- removed the ? at (120.2, 60.5)
- removed the ? at (107.6, 69.2)
- removed the ? at (99.4, 104.7)
- removed the ? at (66.3, 82.0)
- removed the ? at (125.1, 58.1)
- removed the ? at (118.2, 55.6)
- removed the ? at (62.0, 83.2)
- removed the ? at (91.0, 122.0)
- removed the ? at (69.6, 82.3)
- removed the ? at (63.3, 95.5)
- removed the ? at (59.0, 103.0)
- removed the ? at (64.3, 85.3)
- removed the ? at (94.5, 99.0)
- removed the ? at (65.0, 100.1)
- removed the ? at (67.8, 80.0)
- removed the ? at (80.0, 100.0)
- removed the ? at (108.3, 110.6)
- removed the ? at (114.8, 61.1)
- removed the ? at (91.0, 109.0)
- removed the ? at (93.8, 114.5)
- removed the ? at (59.0, 97.0)
- removed the ? at (70.7, 77.5)
- removed the ? at (100.0, 156.0)
- removed the C_BAT at (114.5, 58.0)
- removed the C_BOOST_IN at (113.2, 50.5)
- removed the C_FEEDFORWARD at (117.0, 50.0)
- removed the C_GAUGE at (130.0, 85.5)
- removed the C_KEYS at (97.3, 115.5)
- removed the C_KEYS_BULK at (107.0, 117.0)
- removed the C_LCD_IN at (61.0, 103.0)
- removed the C_LCD_OUT at (61.0, 97.0)
- removed the C_SYS at (123.0, 58.1)
- removed the C_USB at (122.0, 54.9)
- removed the J_BAT at (135.0, 72.0)
- removed the J_LCD at (63.0, 80.0)
- removed the J_OFF at (134.0, 55.0)
- removed the J_USB at (125.0, 43.0)
- removed the L_BOOST at (106.0, 51.0)
- removed the R_ALERT_PULL at (133.0, 85.0)
- removed the R_CC2 at (127.0, 49.0)
- removed the R_CHG_PULL at (125.0, 70.0)
- removed the R_EN at (112.5, 47.0)
- removed the R_FB_HI at (115.5, 53.0)
- removed the R_FB_LO at (115.5, 55.0)
- removed the R_GOOD_PULL at (125.0, 73.0)
- removed the R_ILIM at (126.5, 57.0)
- removed the R_ISET at (114.0, 60.0)
- removed the R_RESET at (106.0, 99.0)
- removed the R_TIMER at (119.0, 53.0)
- removed the SW_A at (134.0, 129.0)
- removed the SW_B at (124.0, 139.0)
- removed the SW_DOWN at (76.0, 139.0)
- removed the SW_LEFT at (66.0, 129.0)
- removed the SW_MENU at (100.0, 142.0)
- removed the SW_RIGHT at (86.0, 129.0)
- removed the SW_SELECT at (88.0, 152.0)
- removed the SW_START at (112.0, 152.0)
- removed the SW_UP at (76.0, 119.0)
- removed the SW_X at (124.0, 119.0)
- removed the SW_Y at (114.0, 129.0)
- removed the TP_5V at (86.0, 53.0)
- removed the TP_GND at (80.0, 53.0)
- removed the U_BOOST at (110.0, 51.0)
- removed the U_CHARGE at (119.0, 58.0)
- removed the U_GAUGE at (132.0, 82.0)
- removed the U_KEYS at (100.0, 108.0)
- removed the U_LCD_PWR at (65.0, 100.0)
- added ?: , tscircuit:g350_mechanical_173ad2003efebb616ac7b73e148e29dd, F.Cu at (135.2, 48.6)
- added ?: , tscircuit:g350_mechanical_188f7ca459ec5b0464b6c69c2359e83c, F.Cu at (107.6, 67.7)
- added ?: , tscircuit:g350_mechanical_1c41598039f833e16fce3ebe1994b15d, F.Cu at (130.5, 48.6)
- added ?: , tscircuit:g350_mechanical_1ea571c02903476133611d023dbef2a3, F.Cu at (124.1, 54.9)
- added ?: , tscircuit:g350_mechanical_24488a20763cd4df37cee0621a256a5d, F.Cu at (124.2, 44.2)
- added ?: , tscircuit:g350_mechanical_271ac4681a4219f85b9ef85863042948, F.Cu at (117.2, 55.7)
- added ?: , tscircuit:g350_mechanical_28f5ac0057b20e3f27a63782590182bd, F.Cu at (100.0, 156.0)
- added ?: , tscircuit:g350_mechanical_2c5d6e4021ff989f17a1c2fe0d43ed5d, F.Cu at (131.3, 52.7)
- added ?: , tscircuit:g350_mechanical_2e1d96183a8617f846ee99d853571bb8, F.Cu at (61.0, 140.0)
- added ?: , tscircuit:g350_mechanical_312e9d54102e410c518b1f6c6d180234, F.Cu at (130.6, 49.5)
- added ?: , tscircuit:g350_mechanical_330a3f404d9d7aff31bacac24eecef7d, F.Cu at (128.0, 85.5)
- added ?: , tscircuit:g350_mechanical_33b335985b54abc815a372d879646e88, F.Cu at (124.8, 47.4)
- added ?: , tscircuit:g350_mechanical_34a222265a65bf3a16925f66787581fa, F.Cu at (125.8, 47.4)
- added ?: , tscircuit:g350_mechanical_38ed92627a4a70c24458b0de02fbd27e, F.Cu at (103.4, 53.8)
- added ?: , tscircuit:g350_mechanical_3c2ff3a071dbc1a11fe776e2320cd3dd, F.Cu at (122.6, 47.7)
- added ?: , tscircuit:g350_mechanical_3cca962849331808559b99e862041bc8, F.Cu at (100.0, 45.0)
- added ?: , tscircuit:g350_mechanical_3da70fa041b136213ef6841e4061c1a3, F.Cu at (67.0, 77.5)
- added ?: , tscircuit:g350_mechanical_403077a04a8e4d4154ec22e25f49f883, F.Cu at (129.2, 83.9)
- added ?: , tscircuit:g350_mechanical_42c3ca406b47eb011953a04238a0aa7d, F.Cu at (127.4, 47.7)
- added ?: , tscircuit:g350_mechanical_05ea26200fd6ec5f2597fede3b59115d, F.Cu at (62.0, 51.0)
- added ?: , tscircuit:g350_mechanical_4590e672043408123d28d64e7e85b4ae, F.Cu at (143.0, 60.0)
- added ?: , tscircuit:g350_mechanical_480707603245f4e11c84e26206c3cfe3, F.Cu at (119.8, 51.7)
- added ?: , tscircuit:g350_mechanical_48e4b000534285a15da05b4267fe30e3, F.Cu at (118.5, 54.5)
- added ?: , tscircuit:g350_mechanical_4a0a79003faca35f354ecdbe2af0f81d, F.Cu at (103.8, 49.5)
- added ?: , tscircuit:g350_mechanical_4b33d1c05591a7615fef7d026a4d52a3, F.Cu at (114.8, 48.7)
- added ?: , tscircuit:g350_mechanical_4c136e803344d7414d62e2fe31f562c3, F.Cu at (112.7, 58.0)
- added ?: , tscircuit:g350_mechanical_4cc2cd32559e704e08005232659f14b2, F.Cu at (62.0, 149.0)
- added ?: , tscircuit:g350_mechanical_08d713c0768132010a26883e7531bd83, F.Cu at (109.0, 48.3)
- added ?: , tscircuit:g350_mechanical_54a590c005caad21603aeb024554d71d, F.Cu at (121.0, 60.0)
- added ?: , tscircuit:g350_mechanical_59c6ecc04fff85df063a07825c7394e3, F.Cu at (135.2, 50.4)
- added ?: , tscircuit:g350_mechanical_5db7e3c00347a5df572898024e672a1d, F.Cu at (117.0, 60.0)
- added ?: , tscircuit:g350_mechanical_5df326a007b9993f4e7ff4225b467e7d, F.Cu at (130.5, 50.4)
- added ?: , tscircuit:g350_mechanical_5f9317604e789de1037bacde556ff79d, F.Cu at (125.2, 44.2)
- added ?: , tscircuit:g350_mechanical_64d7726c2a306ef446c7afac484031b4, F.Cu at (134.5, 82.9)
- added ?: , tscircuit:g350_mechanical_0b9949921801cb72246a4d5230d2cf32, F.Cu at (139.0, 60.0)
- added ?: , tscircuit:g350_mechanical_658cea601b1acfdf643d75e21c6a445d, F.Cu at (67.8, 81.0)
- added ?: , tscircuit:g350_mechanical_66a129e070feff817b5cd5227a45553d, F.Cu at (128.2, 51.0)
- added ?: , tscircuit:g350_mechanical_69a1128073fee8217e5cbdc277456c9d, F.Cu at (126.3, 74.5)
- added ?: , tscircuit:g350_mechanical_6c6d168e78d5986e7ac1e5b26e5963d2, F.Cu at (94.8, 117.0)
- added ?: , tscircuit:g350_mechanical_6d22d3da60ba51fa5451d01a47e94e3a, F.Cu at (80.0, 100.0)
- added ?: , tscircuit:g350_mechanical_774ae8c02e44d95f2c2b648279645d9d, F.Cu at (61.0, 60.0)
- added ?: , tscircuit:g350_mechanical_79ac686006fb51df785cf3e2084ac65d, F.Cu at (120.0, 100.0)
- added ?: , tscircuit:g350_mechanical_7c7c3fe0042b7a5f7b2ccb62057aeedd, F.Cu at (117.0, 56.5)
- added ?: , tscircuit:g350_mechanical_7dc12d8002e68cbf7c71b9020436013d, F.Cu at (123.0, 60.1)
- added ?: , tscircuit:g350_mechanical_08b5d53e03b2aca2101b2e821c83b062, B.Cu at (67.0, 76.3)
- added ?: , tscircuit:g350_mechanical_0beab4205fc5be203489cfa03726a2a0, B.Cu at (69.6, 82.3)
- added ?: , tscircuit:g350_mechanical_140d345c2075b63c2cde381c3946b9fc, B.Cu at (82.0, 113.0)
- added ?: , tscircuit:g350_mechanical_16f4a6202cb5b89f4276cb1e5837dd9d, B.Cu at (118.2, 55.6)
- added ?: , tscircuit:g350_mechanical_188e018e4510c0f25d507c8e004e45f2, B.Cu at (98.8, 104.6)
- added ?: , tscircuit:g350_mechanical_26ba992868177788568baa18152ecbb8, B.Cu at (67.8, 80.0)
- added ?: , tscircuit:g350_mechanical_270478961a9bf6b60e3374d601caf2f6, B.Cu at (96.0, 123.0)
- added ?: , tscircuit:g350_mechanical_27e883326fa77ece073780ce61387d32, B.Cu at (59.0, 97.0)
- added ?: , tscircuit:g350_mechanical_2b4594c437ae16a444169884507f1a64, B.Cu at (59.0, 103.0)
- added ?: , tscircuit:g350_mechanical_2cd810204299229f585a351e6e1b479d, B.Cu at (104.7, 115.5)
- added ?: , tscircuit:g350_mechanical_342a7a08602513b80b8b5e88773bd0c8, B.Cu at (64.3, 85.3)
- added ?: , tscircuit:g350_mechanical_35717a446cefc33c0f5100bc4e4dc1c4, B.Cu at (106.2, 114.5)
- added ?: , tscircuit:g350_mechanical_3a4ca1b8235220c87f0f1cb821705a38, B.Cu at (114.8, 61.1)
- added ?: , tscircuit:g350_mechanical_3de9924042be27ff3c9a1dc2440d9c7d, B.Cu at (62.0, 83.2)
- added ?: , tscircuit:g350_mechanical_405e3ac04abc10615519e6025f77bba3, B.Cu at (63.3, 104.5)
- added ?: , tscircuit:g350_mechanical_459662206430107f0df6831e48430a43, B.Cu at (100.6, 104.7)
- added ?: , tscircuit:g350_mechanical_157764801fd53a212a330fc23490e563, F.Cu at (125.1, 58.1)
- added ?: , tscircuit:g350_mechanical_45b49b202ff388a11a327622047163a3, B.Cu at (107.6, 69.2)
- added ?: , tscircuit:g350_mechanical_4b08715809ab92f837b14b68790e29c8, B.Cu at (66.3, 82.0)
- added ?: , tscircuit:g350_mechanical_4e553ad80cf85c78346481e875c16048, B.Cu at (120.2, 60.5)
- added ?: , tscircuit:g350_mechanical_502d20f643c49f16375c1d362af39b56, B.Cu at (105.5, 99.0)
- added ?: , tscircuit:g350_mechanical_519150505df9d2306a62541076cad5f0, B.Cu at (67.0, 78.8)
- added ?: , tscircuit:g350_mechanical_5309ee6c5f72704c6bdaf22c7843740c, B.Cu at (89.0, 122.0)
- added ?: , tscircuit:g350_mechanical_535e87403d9d74c127dc6242121b4fc3, B.Cu at (125.7, 69.3)
- added ?: , tscircuit:g350_mechanical_5640e24449d860643d6fde8431075ca4, B.Cu at (89.0, 109.0)
- added ?: , tscircuit:g350_mechanical_5e31fa7a009337fa5d0b8a864555b2fa, B.Cu at (91.7, 115.2)
- added ?: , tscircuit:g350_mechanical_67bfaee018e80b5f66703a621a377fdd, B.Cu at (65.0, 99.9)
- added ?: , tscircuit:g350_mechanical_1710d3a0684772211860481e66f7fda3, F.Cu at (139.0, 140.0)
- added ?: , tscircuit:g350_mechanical_68c15ecc399fdeb423fee3cc7e6259b4, B.Cu at (94.3, 115.2)
- added ?: , tscircuit:g350_mechanical_6916d64012dd48df435c4482666a2e1d, B.Cu at (107.0, 115.8)
- added ?: , tscircuit:g350_mechanical_694cd88c5ce456ac507bd4cc441352ec, B.Cu at (82.0, 104.0)
- added ?: , tscircuit:g350_mechanical_6f83ba72280c478e4063b672572c4b8e, B.Cu at (66.0, 84.0)
- added ?: , tscircuit:g350_mechanical_765b7ac07f46af9f74e8d9fe6a8b045d, B.Cu at (68.6, 82.8)
- added ?: , tscircuit:g350_mechanical_7bd6d8ba1026667a5b8a0bc638c581fa, B.Cu at (90.5, 116.0)
- added ?: , tscircuit:g350_mechanical_7cf5d8e0114566a05a6b0ba039e48220, B.Cu at (67.7, 83.4)
- added C_BAT: 10uF, tscircuit:g350_C_BAT_47d06ae03787dae1491fdf5e36386663, F.Cu at (114.5, 58.0)
- added C_BOOST_IN: 10uF, tscircuit:g350_C_BOOST_IN_5255146047f73ebf3d99691e333b937d, F.Cu at (113.2, 50.5)
- added C_FEEDFORWARD: 220pF, tscircuit:g350_C_FEEDFORWARD_16c584a07135c2813459ff9e26163e43, F.Cu at (117.0, 50.0)
- added C_GAUGE: 100nF, tscircuit:g350_C_GAUGE_07aee08077a9654108fe54fe7659f0c3, F.Cu at (130.0, 85.5)
- added C_KEYS: 100nF, tscircuit:g350_C_KEYS_644960c23e17dcbe1f86e5c27d25a842, F.Cu at (102.7, 115.5)
- added C_KEYS_BULK: 10uF, tscircuit:g350_C_KEYS_BULK_468ee6ca3a2664ea2dbde30a2155612a, F.Cu at (93.0, 117.0)
- added C_LCD_IN: 1uF, tscircuit:g350_C_LCD_IN_5be2f4460c8d09ba74fd07ba2292fa46, F.Cu at (61.0, 97.0)
- added C_LCD_OUT: 1uF, tscircuit:g350_C_LCD_OUT_796ff1802c1fd09f2e506d42773f54dd, F.Cu at (61.0, 103.0)
- added C_SYS: 10uF, tscircuit:g350_C_SYS_08f8654077af54ff07a8f0c278fec97d, F.Cu at (123.0, 58.1)
- added C_USB: 1uF, tscircuit:g350_C_USB_6f7d3200112a883f6e2dbd821279fcbd, F.Cu at (122.0, 54.9)
- added C_USB_ESD: 100nF, tscircuit:g350_C_USB_ESD_55af1c004fe0a61f0a8f97c264ffd5a3, F.Cu at (129.0, 52.0)
- added J_BAT: J_BAT, tscircuit:g350_J_BAT_1c1b67e03e54d601673aec1e0ccaae3d, F.Cu at (135.0, 72.0)
- added J_LCD: FPC-05F-18PH20, tscircuit:g350_J_LCD_023284580e9b06381b038818276c09f8, F.Cu at (66.2, 80.0)
- added J_OFF: J_OFF, tscircuit:g350_J_OFF_72356f40335a52df2715eb027e79d71d, F.Cu at (134.0, 55.0)
- added J_USB: TYPE-C-31-M-12, tscircuit:g350_J_USB_2a17ef222ac30dde7f9e0ade2b86f822, F.Cu at (125.0, 43.0)
- added J_USB_LINK: J_USB_LINK, tscircuit:g350_J_USB_LINK_151b40200abd6a7f005f94de09fe40c3, F.Cu at (144.5, 48.5)
- added L_BOOST: 1µH, tscircuit:g350_L_BOOST_162d00c0709d3ea134f2837e257dba63, F.Cu at (106.0, 51.0)
- added R_ALERT_PULL: 100kΩ, tscircuit:g350_R_ALERT_PULL_3ed784801b98b9617608f7422f86cadd, F.Cu at (133.0, 85.0)
- added R_CC1: 5.1kΩ, tscircuit:g350_R_CC1_1675a34070e5e12134a9e0fe25c65ce3, F.Cu at (127.0, 49.0)
- added R_CHG_PULL: 100kΩ, tscircuit:g350_R_CHG_PULL_7cb2e42028dcddff31935fe273fc623d, F.Cu at (125.0, 70.0)
- added R_EN: 100kΩ, tscircuit:g350_R_EN_2bedbaa0536a8b212d3d2f1e521b16a3, F.Cu at (112.5, 47.0)
- added R_FB_HI: 732kΩ, tscircuit:g350_R_FB_HI_577e14c02929a57f562ea0422a7919fd, F.Cu at (115.5, 53.0)
- added R_FB_LO: 100kΩ, tscircuit:g350_R_FB_LO_1fea8fa05f6db621213a041e5e1e41a3, F.Cu at (115.5, 55.0)
- added R_GOOD_PULL: 100kΩ, tscircuit:g350_R_GOOD_PULL_2f2dc0202b427dc17a4d445e1fdd067d, F.Cu at (125.0, 73.0)
- added R_ILIM: 3.3kΩ, tscircuit:g350_R_ILIM_21d596405ed223ff208621c26021987d, F.Cu at (126.5, 57.0)
- added R_ISET: 3.3kΩ, tscircuit:g350_R_ISET_2238e4a07ca9228128e69f9e31899e43, F.Cu at (114.0, 60.0)
- added R_RESET: 10kΩ, tscircuit:g350_R_RESET_1a8653a074f691813099309e29d70d43, F.Cu at (94.0, 99.0)
- added R_TIMER: 68kΩ, tscircuit:g350_R_TIMER_7999bf001f29811f3b46bcc26a49055d, F.Cu at (119.0, 53.0)
- added R_USB_EN1: 100kΩ, tscircuit:g350_R_USB_EN1_2d820ae02cee330178a18f1e1e31513d, F.Cu at (108.0, 81.0)
- added R_USB_EN2: 100kΩ, tscircuit:g350_R_USB_EN2_18011b8072715961331e68be2751d523, F.Cu at (108.0, 84.0)
- added SW_A: SW_A, tscircuit:g350_SW_A_69607ec017473b7f68110a421896affd, F.Cu at (134.0, 129.0)
- added SW_B: SW_B, tscircuit:g350_SW_B_732329a00c351c2174729e1e0ae5a7a3, F.Cu at (124.0, 139.0)
- added SW_DOWN: SW_DOWN, tscircuit:g350_SW_DOWN_66fbc8fa73644ada7fccccba73cab166, F.Cu at (76.0, 139.0)
- added SW_LEFT: SW_LEFT, tscircuit:g350_SW_LEFT_093028fc1598aadc22012cbc2e69ae9c, F.Cu at (66.0, 129.0)
- added SW_MENU: SW_MENU, tscircuit:g350_SW_MENU_4553bc603b53fddf440447e23ca3725d, F.Cu at (100.0, 142.0)
- added SW_RIGHT: SW_RIGHT, tscircuit:g350_SW_RIGHT_2a1c1df636849fd642ed21b64f55a396, F.Cu at (86.0, 129.0)
- added SW_SELECT: SW_SELECT, tscircuit:g350_SW_SELECT_69cf658e5d66e3ae50fe61ce4495dfee, F.Cu at (88.0, 152.0)
- added SW_START: SW_START, tscircuit:g350_SW_START_4c2facc034780d7f4ae0384235c781fd, F.Cu at (112.0, 152.0)
- added SW_UP: SW_UP, tscircuit:g350_SW_UP_0f36f6001b9f77e02807f9c034707ba0, F.Cu at (76.0, 119.0)
- added SW_X: SW_X, tscircuit:g350_SW_X_35f9e5604aadd4df34aa70e24bfd495d, F.Cu at (124.0, 119.0)
- added SW_Y: SW_Y, tscircuit:g350_SW_Y_59763d0027317d3f5826c8822880f1bd, F.Cu at (114.0, 129.0)
- added TP_5V: TP_5V, tscircuit:g350_TP_5V_19c1e4e0743222c1315d9f5e29129e83, F.Cu at (86.0, 53.0)
- added TP_GND: TP_GND, tscircuit:g350_TP_GND_1bb7c0407627fe212f67c3fe2b0879e3, F.Cu at (80.0, 53.0)
- added U_BOOST: TPS61023DRLR, tscircuit:g350_U_BOOST_1f3f53c079af91a12be0307e2e900d63, F.Cu at (110.0, 51.0)
- added U_CHARGE: BQ24074RGTR, tscircuit:g350_U_CHARGE_5486e04005e95da160599b824536269d, F.Cu at (119.0, 58.0)
- added U_GAUGE: MAX17048G+T10, tscircuit:g350_U_GAUGE_1b637ee075d3bcc12fbc055e2ab43883, F.Cu at (132.0, 82.0)
- added U_KEYS: MCP23017-E/SO, tscircuit:g350_U_KEYS_647741a01ae1042165c6b61e19918fa3, F.Cu at (100.0, 108.0)
- added U_LCD_PWR: AP2112K-3.3TRG1, tscircuit:g350_U_LCD_PWR_6bb0e2e01140a4ff492f98e25c60293d, F.Cu at (65.0, 100.0)
- added U_USB_ESD: USBLC6-2SC6, tscircuit:g350_U_USB_ESD_7ae7b8e0673f34e15396b0e23fee2ce3, F.Cu at (133.0, 49.5)
- C_BOOST_OUT1: footprint tscircuit:g350_C_BOOST_OUT1_4c2ad4da72784cc6311b6e6610416ffa -> tscircuit:g350_C_BOOST_OUT1_7e38f91c406a288400f2b5dc424f943c
- C_BOOST_OUT2: footprint tscircuit:g350_C_BOOST_OUT2_7361d6200bf66fa174b14a9e0aa6fb23 -> tscircuit:g350_C_BOOST_OUT2_1b885d80651f5cbf1a38e902666ed13d
- J_PI, J_SPEAKER: moved to F.Cu
- R_CC2: renamed from R_CC1; footprint tscircuit:g350_R_CC1_70956ae034fa573f2575e6a27fe62483 -> tscircuit:g350_R_CC2_70956ae034fa573f2575e6a27fe62483
- TP_3V3: footprint tscircuit:g350_TP_3V3_28035840326ce5a17322dc7e18b29e9d -> tscircuit:g350_TP_3V3_7afe24202a919dff2fde9fe275b1223d; moved to F.Cu
- turned J_SPEAKER to 180 degrees
- turned R_CC2 to 180 degrees
Connections:
- J_PI pad 18: (no net) -> USB_EN1
- J_PI pad 36: (no net) -> USB_EN2
- R_CC2 pad 1: R_CC1.pin1 to J_USB.CC1 -> J_USB.CC2 to R_CC2.pin1
Routing:
- net USB_EN2: track 0.00 -> 68.4 mm, vias 0 -> 3
- net USB_EN1: track 0.00 -> 35.9 mm, vias 0 -> 1
- net USB_DP: track 0.00 -> 24.4 mm, vias 0 -> 4
- net USB_DN: track 0.00 -> 24.3 mm, vias 0 -> 4
- net BUTTON_MENU: track 51.3 -> 28.9 mm
- net SW_X.pin1 to U_KEYS.GPA6: track 20.7 -> 39.6 mm, vias 1 -> 2
- net SDA: track 202.4 -> 184.3 mm, vias 6 -> 8
- net SW_A.pin1 to U_KEYS.GPA4: track 39.0 -> 52.4 mm, vias 1 -> 4
- net SW_B.pin1 to U_KEYS.GPA5: track 41.1 -> 52.8 mm, vias 1 -> 2
- net V5V: track 416.8 -> 405.9 mm, vias 11 -> 12
- net SCL: track 184.9 -> 174.5 mm
- net V3V3: track 335.6 -> 325.2 mm
- net USB_5V: track 19.5 -> 29.7 mm, vias 1 -> 5
- net SW_RIGHT.pin1 to U_KEYS.GPA3: track 39.9 -> 29.9 mm, vias 4 -> 2
- net V_LCD3V3: track 33.2 -> 42.8 mm
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Other:
- board text added: "G350 LINUX / REV B"
- board text added: "USB LINK"
- board text added: "USB-C"
- board text removed: "G350 LINUX / REV A"
