File: fabrication/kicad/index.kicad_sch (KiCad schematic)
At the start: 130 parts

Commit message: Release top-only Rev B carrier with shared USB-C charging and data
Parts:
- removed GND (x50): GND, symbol Custom:rail_down
- removed USB_5V: USB_5V, symbol Custom:rail_up
- removed V3V3 (x6): V3V3, symbol Custom:rail_up
- removed V5V (x9): V5V, symbol Custom:rail_up
- removed VBAT (x3): VBAT, symbol Custom:rail_up
- removed VSYS (x4): VSYS, symbol Custom:rail_up
- removed V_LCD3V3 (x2): V_LCD3V3, symbol Custom:rail_up
- added C_USB_ESD: 100nF, symbol Device:capacitor_down
- added GND (x55): GND, symbol Custom:rail_down
- added J_USB_LINK: J_USB_LINK, symbol Connector_Generic:Conn_01x3_J_USB_LINK
- added R_USB_EN1, R_USB_EN2: 100kΩ, symbol Device:boxresistor_down
- added USB_5V (x2): USB_5V, symbol Custom:rail_up
- added U_USB_ESD: USBLC6-2SC6, symbol Device:U_USBLC6-2SC6
- added V3V3 (x6): V3V3, symbol Custom:rail_up
- added V5V (x9): V5V, symbol Custom:rail_up
- added VBAT (x3): VBAT, symbol Custom:rail_up
- added VSYS (x4): VSYS, symbol Custom:rail_up
- added V_LCD3V3 (x2): V_LCD3V3, symbol Custom:rail_up
Connections:
- net VSYS: no longer U_CHARGE.6 (EN1)
- net at U_AUDIO.11 (GND2), U_AUDIO.15 (GND3), U_AUDIO.17 (EP): now also GND.1
- net at U_AUDIO.3 (GND1): now also GND.1
- net at SW_DOWN.2: now also GND.1
- net at SW_RIGHT.2: now also GND.1
- net at U_BOOST.6 (VOUT): now also V5V.1
- net at TP_5V.1: now also V5V.1
- net at SW_START.2: now also GND.1
- net at C_AUDIO_HF.2: now also GND.1
- net at R_AUDIO_PD.2: now also GND.1
- net at U_CHARGE.2 (BAT1), U_CHARGE.3 (BAT2): now also VBAT.1
- net at C_LCD_OUT.1, U_LCD_PWR.5 (VOUT): now also V_LCD3V3.1
- net at C_LCD_OUT.2: now also GND.1
- net at C_LCD_IN.2: now also GND.1
- net at R_FB_LO.2: now also GND.1
- net at C_KEYS_BULK.1: now also V3V3.1
- net at R_CHG_PULL.1, R_GOOD_PULL.1: now also V3V3.1
- net at J_USB.1 (EH2), J_USB.13 (A1B12), J_USB.14 (B1A12)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: now also GND.1
- net J_USB_B5: now reaches J_USB.12 (B5)
- net J_USB_B5: now also R_CC2.1
- net at J_PI.1 (J8_1), TP_3V3.1: now also V3V3.1
- net at J_PI.2 (J8_2), J_PI.4 (J8_4): now also V5V.1
- net at J_PI.25 (J8_25), J_PI.30 (J8_30), J_PI.34 (J8_34)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: now also GND.1
- net at SW_MENU.2: now also GND.1
- net at C_BAT.1, C_GAUGE.1: now also VBAT.1
- net at C_GAUGE.2: now also GND.1
- net at J_LCD.1, J_LCD.10: now also V_LCD3V3.1
- net at J_LCD.19, J_LCD.20: now also GND.1
- net at J_LCD.3: now also GND.1
- net at U_BOOST.3 (VIN): now also VSYS.1
- net at U_GAUGE.1 (CTG), U_GAUGE.4 (GND): now also GND.1
- net at U_GAUGE.6 (QSTRT), U_GAUGE.9 (EP): now also GND.1
- net at J_BAT.1: now also VBAT.1
- net at J_BAT.2: now also GND.1
- net at C_BOOST_IN.1, C_SYS.1: now also VSYS.1
- net at C_BOOST_IN.2: now also GND.1
- net at R_ISET.2: now also GND.1
- net at C_USB.1: now also C_USB_ESD.1, USB_5V.1; no longer U_CHARGE.13 (IN)
- net at C_AUDIO_BULK.2: now also GND.1
- net at R_TIMER.2: now also GND.1
- net at R_CC1.2: now also GND.1
- net at U_KEYS.10 (VSS): now also GND.1
- net at SW_X.2: now also GND.1
- net at J_OFF.2: now also GND.1
- net at U_LCD_PWR.1 (VIN), U_LCD_PWR.3 (EN): now also V5V.1
- net at U_CHARGE.8 (VSS): now also GND.1
- net at SW_B.2: now also GND.1
- net at C_SYS.2: now also GND.1
- net at C_BAT.2: now also GND.1
- net at U_KEYS.15 (A0), U_KEYS.16 (A1), U_KEYS.17 (A2): now also GND.1
- net at C_LCD_IN.1: now also V5V.1
- net at C_BOOST_OUT1.1, C_BOOST_OUT2.1: now also V5V.1
- net at C_BOOST_OUT2.2: now also GND.1
- net at SW_A.2: now also GND.1
- net at U_BOOST.4 (GND): now also GND.1
- net at C_AUDIO_BULK.1, C_AUDIO_HF.1: now also V5V.1
- net at C_USB.2: now also GND.1
- net at R_CC2.2: now also GND.1
- net at R_ALERT_PULL.1: now also V3V3.1
- net at U_CHARGE.17 (EP): now also GND.1
- net at U_CHARGE.4 (N_CE): now also GND.1; no longer U_CHARGE.5 (EN2)
- net at C_KEYS_BULK.2: now also GND.1
- net at U_LCD_PWR.2 (GND): now also GND.1
- net at C_KEYS.1: now also V3V3.1
- net at C_KEYS.2: now also GND.1
- net at C_FEEDFORWARD.1, R_FB_HI.1: now also V5V.1
- net at C_BOOST_OUT1.2: now also GND.1
- net at R_EN.1: now also VSYS.1
- net at SW_LEFT.2: now also GND.1
- net at R_RESET.2, U_KEYS.9 (VDD): now also V3V3.1
- net at L_BOOST.1: now also VSYS.1
- net at TP_GND.1: now also GND.1
- net at R_ILIM.2: now also GND.1
- net at SW_UP.2: now also GND.1
- net at SW_SELECT.2: now also GND.1
- net at SW_Y.2: now also GND.1
- new net: C_USB_ESD.2, GND.1
- new net: GND.1, R_USB_EN2.2
- new net: USB_5V.1, U_CHARGE.13 (IN), U_USB_ESD.5
- new net: R_USB_EN1.1, U_CHARGE.6 (EN1)
- new net: GND.1, U_USB_ESD.2
- new net: GND.1, J_USB_LINK.3
- new net: GND.1, R_USB_EN1.2
Other:
- note added: "Controls / MCP23017 0x20"
- note added: "USB_DN"
- note added: "USB_DP"
- note added: "USB_EN1"
- note added: "USB_EN2"
- note removed: "Front controls — MCP23017 address 0x20"
- note removed: "USB_CC2"
